File: kicad_6502/kicad_6502.kicad_sch (KiCad schematic)
At the start: 47 parts, among them J1 A[3...0], J10 TX, J11 RX, J12 IX0, J13 IX1, J14 EXT, J2 D[7...0], J3 R/W, J4 /NMI, J5 PORTA, J6 PORTB, J7 CA, J8 CB, J9 RXC, SW1 RESET, U1 CPU, U2 ACIA, U3 VIA, U4 SRAM, U5 ROM, U6 74LS08, U7 ATF22V10C, U8 74LS73, Y1 4MHz, Y2 1.8432MHz

Commit message: schimbari kicad
Parts:
- removed C10: 100nF, Capacitor_THT:C_Disc_D3.0mm_W2.0mm_P2.50mm, symbol Device:C_Small
- removed C11: 47uF, Capacitor_THT:CP_Radial_D5.0mm_P2.50mm, symbol Device:C_Polarized_Small
- removed J1: A[3...0], Connector_PinHeader_2.54mm:PinHeader_1x04_P2.54mm_Vertical, symbol Connector_Generic:Conn_01x04
- removed J13: IX1, Connector_PinHeader_2.54mm:PinHeader_1x01_P2.54mm_Vertical, symbol Connector_Generic:Conn_01x01
- removed J14: EXT, Connector_PinHeader_2.54mm:PinHeader_1x02_P2.54mm_Vertical, symbol Connector_Generic:Conn_01x02
- removed J2: D[7...0], Connector_PinHeader_2.54mm:PinHeader_1x08_P2.54mm_Vertical, symbol Connector_Generic:Conn_01x08
- removed J3: R/W, Connector_PinHeader_2.54mm:PinHeader_1x01_P2.54mm_Vertical, symbol Connector_Generic:Conn_01x01
- removed J4: /NMI, Connector_PinHeader_2.54mm:PinHeader_1x01_P2.54mm_Vertical, symbol Connector_Generic:Conn_01x01
- removed U2: ACIA, Package_DIP:DIP-28_W15.24mm, symbol PCM_65xx-library:W65C51NxP
- removed U3: VIA, Package_DIP:DIP-40_W15.24mm, symbol PCM_65xx-library:W65C22NxP
- removed U4: SRAM, Package_DIP:DIP-28_W15.24mm, symbol Memory_RAM:KM62256CLP
- removed U5: ROM, Package_DIP:DIP-28_W15.24mm, symbol Memory_EEPROM:28C256
- removed U6: 74LS08, Package_DIP:DIP-14_W7.62mm, symbol 74xx:74LS08
- removed U7: ATF22V10C, Package_DIP:DIP-24_W7.62mm, symbol ATF:ATF22V10C-15PU
- removed U8: 74LS73, Package_DIP:DIP-14_W7.62mm, symbol 74xx:74LS73
- added C10: 4.7uF, Capacitor_THT:CP_Radial_D5.0mm_P2.50mm, symbol Device:C_Polarized_Small
- added J1: /IRQ, Connector_PinHeader_2.54mm:PinHeader_1x01_P2.54mm_Vertical, symbol Connector_Generic:Conn_01x01
- added J13: PWR, Connector_PinHeader_2.54mm:PinHeader_1x02_P2.54mm_Vertical, symbol Connector_Generic:Conn_01x02
- added J2: /NMI, Connector_PinHeader_2.54mm:PinHeader_1x01_P2.54mm_Vertical, symbol Connector_Generic:Conn_01x01
- added J3: D[7...0], Connector_PinHeader_2.54mm:PinHeader_1x08_P2.54mm_Vertical, symbol Connector_Generic:Conn_01x08
- added J4: A[3...0], Connector_PinHeader_2.54mm:PinHeader_1x04_P2.54mm_Vertical, symbol Connector_Generic:Conn_01x04
- added U2: EEPROM, Package_DIP:DIP-28_W15.24mm, symbol Memory_EEPROM:28C256
- added U3: SRAM, Package_DIP:DIP-28_W15.24mm, symbol Memory_RAM:CY62256-70PC
- added U4: ACIA, Package_DIP:DIP-28_W15.24mm, symbol PCM_65xx-library:W65C51NxP
- added U5: VIA, Package_DIP:DIP-40_W15.24mm, symbol PCM_65xx-library:W65C22NxP
- added U6: ATF22V10, Package_DIP:DIP-24_W7.62mm, symbol 2026-05-11_16-07-16:ATF22V10C-15PU
- added U7: 74LS73, Package_DIP:DIP-14_W7.62mm, symbol 74xx:74LS73
- C1, C2, C3, C4, C5, C6, C7, C8, C9: value 100nF -> 0.1uF; footprint Capacitor_THT:C_Disc_D3.0mm_W2.0mm_P2.50mm -> Capacitor_THT:C_Disc_D3.4mm_W2.1mm_P2.50mm
- J10: value TX -> /IRQ_ACIA
- J11: value RX -> TX
- J12: value IX0 -> RX
- J5: value PORTA -> PORTB
- J6: value PORTB -> PORTA
- J9: value RXC -> /IRQ_VIA
- R1, R11, R2, R3, R4, R5, R6, R7, R8: footprint Resistor_THT:R_Axial_DIN0207_L6.3mm_D2.5mm_P2.54mm_Vertical -> Resistor_THT:R_Axial_DIN0207_L6.3mm_D2.5mm_P7.62mm_Horizontal
- R10: value 20K -> 250K; footprint Resistor_THT:R_Axial_DIN0207_L6.3mm_D2.5mm_P2.54mm_Vertical -> Resistor_THT:R_Axial_DIN0207_L6.3mm_D2.5mm_P7.62mm_Horizontal
- R9: value 20K -> 5K; footprint Resistor_THT:R_Axial_DIN0207_L6.3mm_D2.5mm_P2.54mm_Vertical -> Resistor_THT:R_Axial_DIN0207_L6.3mm_D2.5mm_P7.62mm_Horizontal
- Y1: value 4MHz -> SYS_CLK
- Y2: value 1.8432MHz -> COM_CLK
Connections:
- net +5V: now also J13.1 (Pin_1), U2.27 (~{WE}), U2.28 (VCC), U3.28 (VCC), U4.15 (VCC), U5.20 (VCC), U6.24 (VCC), U7.10 (K), U7.14 (J), U7.4 (VCC), U7.5 (C), U7.6 (~{R}), U7.7 (J); no longer J12.1 (Pin_1)
- net A0: now also J4.1 (Pin_1), U2.10 (A0), U3.10 (A0), U4.14 (RS1), U5.38 (RS0)
- net A1: now also J4.2 (Pin_2), U2.9 (A1), U3.9 (A1), U4.13 (RS0), U5.37 (RS1)
- net A10: now also U2.21 (A10), U3.21 (A10), U6.6 (IN)
- net A11: now also U2.23 (A11), U3.23 (A11), U6.5 (IN)
- net A12: now also U2.2 (A12), U3.2 (A12), U6.4 (IN/PD)
- net A13: now also U2.26 (A13), U3.26 (A13), U6.3 (IN)
- net A14: now also U2.1 (A14), U3.1 (A14), U6.2 (IN)
- net A15: now also U6.1 (CLK/IN)
- net A2: now also J4.3 (Pin_3), U2.8 (A2), U3.8 (A2), U5.36 (RS2)
- net A3: now also J4.4 (Pin_4), U2.7 (A3), U3.7 (A3), U5.35 (RS3)
- net A4: now also U2.6 (A4), U3.6 (A4), U6.13 (IN)
- net A5: now also U2.5 (A5), U3.5 (A5), U6.11 (IN)
- net A6: now also U2.4 (A6), U3.4 (A6), U6.10 (IN)
- net A7: now also U2.3 (A7), U3.3 (A7), U6.9 (IN)
- net A8: now also U2.25 (A8), U3.25 (A8), U6.8 (IN)
- net A9: now also U2.24 (A9), U3.24 (A9), U6.7 (IN)
- net D0: now also J3.1 (Pin_1), U2.11 (D0), U3.11 (Q0), U4.18 (D0), U5.33 (D0)
- net D1: now also J3.2 (Pin_2), U2.12 (D1), U3.12 (Q1), U4.19 (D1), U5.32 (D1)
- net D2: now also J3.3 (Pin_3), U2.13 (D2), U3.13 (Q2), U4.20 (D2), U5.31 (D2)
- net D3: now also J3.4 (Pin_4), U2.15 (D3), U3.15 (Q3), U4.21 (D3), U5.30 (D3)
- net D4: now also J3.5 (Pin_5), U2.16 (D4), U3.16 (Q4), U4.22 (D4), U5.29 (D4)
- net D5: now also J3.6 (Pin_6), U2.17 (D5), U3.17 (Q5), U4.23 (D5), U5.28 (D5)
- net D6: now also J3.7 (Pin_7), U2.18 (D6), U3.18 (Q6), U4.24 (D6), U5.27 (D6)
- net D7: now also J3.8 (Pin_8), U2.19 (D7), U3.19 (Q7), U4.25 (D7), U5.26 (D7)
- net GNDD: now also C10.2, J13.2 (Pin_2), U2.14 (GND), U3.14 (GND), U4.1 (VSS), U5.1 (VSS), U6.12 (GND), U7.11 (GND), U7.3 (K)
- net R/W: now also U4.28 (R/~{W}), U5.22 (R/~{W}), U6.14 (I/O)
- net /CE_ROM: now also U2.20 (~{CS}), U2.22 (~{OE}), U6.21 (I/O)
- net /RESET: now also U4.4 (~{RES}), U5.34 (~{RES}), U7.12 (Q)
- net at J6.1 (Pin_1): now also U5.10 (PB0)
- net at J6.2 (Pin_2): now also U5.11 (PB1)
- net at J6.3 (Pin_3): now also U5.12 (PB2)
- net at J6.4 (Pin_4): now also U5.13 (PB3)
- net at J6.5 (Pin_5): now also U5.14 (PB4)
- net at J6.6 (Pin_6): now also U5.15 (PB5)
- net at J6.7 (Pin_7): now also U5.16 (PB6)
- net at J6.8 (Pin_8): now also U5.17 (PB7)
- net at J8.1 (Pin_1): now also U5.18 (CB1)
- net at J8.2 (Pin_2): now also U5.19 (CB2)
- net at J5.1 (Pin_1): now also U5.2 (PA0)
- net at J5.2 (Pin_2): now also U5.3 (PA1)
- net at J7.2 (Pin_2): now also U5.39 (CA2)
- net at J5.3 (Pin_3): now also U5.4 (PA2)
- net at J7.1 (Pin_1): now also U5.40 (CA1)
- net at J5.4 (Pin_4): now also U5.5 (PA3)
- net at J5.5 (Pin_5): now also U5.6 (PA4)
- net at J5.6 (Pin_6): now also U5.7 (PA5)
- net at J5.7 (Pin_7): now also U5.8 (PA6)
- net at J5.8 (Pin_8): now also U5.9 (PA7)
- net at U1.36 (BE): now also R2.2; no longer R4.2
- net at R11.2: now also R10.1, C10.1
- net at J11.1 (Pin_1): now also U4.10 (TxD)
- net at R10.2: now also R9.2, SW1.2; no longer R11.1
- net at U1.2 (RDY): now also R3.2; no longer R1.2
- net at J10.1 (Pin_1): now also R8.2, U4.26 (~{IRQ})
- net at U1.6 (~{NMI}): now also R4.2, J2.1 (Pin_1); no longer R2.2
- net at R6.2: now also U4.2 (CS1)
- net at J9.1 (Pin_1): now also U5.21 (~{IRQ})
- net at U1.7 (SYNC): no longer R3.2
- net at R7.2: now also U5.24 (CS1)
- net at U1.38 (~{SO}): now also R1.2; no longer R5.2
- net CLK_COM renamed COM_CLK
- net COM_CLK: now also U4.6 (XTAL1)
- net CLK_SYS renamed SYS_CLK
- net SYS_CLK: now also U4.27 (ϕ2), U5.25 (ϕ2), U6.15 (I/O), U7.1 (C)
- net IRQ_CPU: no longer names the net of U1.4 (~{IRQ})
- net IRQ_CPU: now also R5.2, J1.1 (Pin_1)
- new net: R11.1, U7.2 (~{R})
- new net: J12.1 (Pin_1), U4.12 (RxD)
- new net /CE_ACIA: U4.3 (~{CS2}), U6.17 (I/O)
- new net /CE_RAM: U3.20 (~{CS}), U6.20 (I/O)
- new net /CE_VIA: U5.23 (~{CS2}), U6.16 (I/O)
- new net /OE_RAM: U3.22 (~{OE}), U6.19 (I/O)
- new net /WE_RAM: U3.27 (~{WE}), U6.18 (I/O)
- no-connect marks 13 -> 17
Other:
- title: Microcalculator -> (none)
